File: APRS_TRACKER_OLED_DAC.kicad_pcb (KiCad board)
At the start: 2 copper layers, 52.6 x 40 mm, 40 parts, among them J1 PWR_IN, J2 ICSP, J3 OLED Conn, J4 Radio Conn, J5 GPS Module, J9 PTT Shunt, Q1 SS8050, U1 ATMEGA328PB-AU, U2 MCP1703Ax-500xxDB, Y1 16MHz

Commit message: Moved ATMEGA library to proper location. Made some adjustments to ISP and DAC pin connections.
Connections:
- net /RST renamed /RESET
- J2 pad 4: /MOSI -> /B3
- J9 pad 2: /PTT -> Net-(J9-Pin_2)
- Q1 pad 3: Net-(Q1-C) -> /PTT
- R13 pad 1: /SD -> /SQL
- R3 pad 1: /PTT -> /TX_EN
- R4 pad 2: /PTT -> /TX_EN
- R7 pad 1: /PTT -> Net-(J9-Pin_2)
- R7 pad 2: Net-(Q1-C) -> /PTT
- U1 pad 19: /B2 -> unconnected-(U1-PE2(ADC6/PTCY/ICP3/~{SS1})-Pad19)
- U1 pad 2: /PTT -> /TX_EN
- U1 pad 22: /B3 -> unconnected-(U1-PE3(ADC7/PTCY/T3/MOSI1)-Pad22)
- U1 pad 23: unconnected-(U1-PC0(ADC0/PTCY/MISO1)-Pad23) -> /B0
- U1 pad 24: unconnected-(U1-PC1(ADC1/PTCY/SCK1)-Pad24) -> /B1
- U1 pad 25: unconnected-(U1-PC2(ADC2/PTCY)-Pad25) -> /B2
- U1 pad 26: /SD -> /B3
- U1 pad 3: /B0 -> unconnected-(U1-PE0(SDA1/ICP4/ACO/PTCXY)-Pad3)
- U1 pad 31: /AUDIO_IN -> /SQL
- U1 pad 6: /B1 -> unconnected-(U1-PE1(SCL1/T4/PTCXY)-Pad6)
Changed lines of the file:
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@@
 	(net 4 "/XTAL1")
 	(net 5 "/XTAL2")
-	(net 6 "/AUDIO_IN")
+	(net 6 "/RESET")
 	(net 7 "Net-(Q1-B)")
 	(net 8 "Net-(C7-Pad2)")
@@
 	(net 14 "/SDA")
 	(net 15 "/MISO")
-	(net 16 "/RST")
+	(net 16 "Net-(J9-Pin_2)")
 	(net 17 "/SCK")
 	(net 18 "/GPS_RXD")
@@
 	(net 23 "/CTRL_0")
 	(net 24 "/CTRL_1")
-	(net 25 "unconnected-(U1-PC0(ADC0{slash}PTCY{slash}MISO1)-Pad23)")
-	(net 26 "unconnected-(U1-PC2(ADC2{slash}PTCY)-Pad25)")
+	(net 25 "/TX_EN")
+	(net 26 "/SQL")
 	(net 27 "unconnected-(U1-PB2(~{SS0}{slash}OC1B{slash}PTCXY)-Pad14)")
 	(net 28 "unconnected-(U1-AREF-Pad20)")
@@
 	(net 30 "unconnected-(U1-PB1(OC1A{slash}PTCXY)-Pad13)")
 	(net 31 "Net-(D4-A)")
-	(net 32 "unconnected-(U1-PC1(ADC1{slash}PTCY{slash}SCK1)-Pad24)")
+	(net 32 "unconnected-(U1-PE2(ADC6{slash}PTCY{slash}ICP3{slash}~{SS1})-Pad19)")
 	(net 33 "/MOSI")
 	(net 34 "/B0")
@@
 	(net 38 "/B3")
 	(net 39 "Net-(R12-Pad1)")
-	(net 40 "/SD")
-	(net 41 "Net-(Q1-C)")
+	(net 40 "unconnected-(U1-PE1(SCL1{slash}T4{slash}PTCXY)-Pad6)")
+	(net 41 "unconnected-(U1-PE3(ADC7{slash}PTCY{slash}T3{slash}MOSI1)-Pad22)")
 	(net 42 "Net-(C8-Pad1)")
 	(net 43 "/SQL_SET")
 	(net 44 "/CD_SQL")
+	(net 45 "unconnected-(U1-PE0(SDA1{slash}ICP4{slash}ACO{slash}PTCXY)-Pad3)")
 	(footprint "LED_SMD:LED_0805_2012Metric_Pad1.15x1.40mm_HandSolder"
 		(layer "F.Cu")
@@
 			(layers "*.Cu" "*.Mask")
 			(remove_unused_layers no)
-			(net 33 "/MOSI")
+			(net 38 "/B3")
 			(pinfunction "Pin_4")
 			(pintype "passive")
@@
 			(layers "*.Cu" "*.Mask")
 			(remove_unused_layers no)
-			(net 16 "/RST")
+			(net 6 "/RESET")
 			(pinfunction "Pin_5")
 			(pintype "passive")
@@
 			(layers "F.Cu" "F.Mask" "F.Paste")
 			(roundrect_rratio 0.208333)
-			(net 40 "/SD")
+			(net 26 "/SQL")
 			(pintype "passive")
 		)
@@
 			(size 1.6 0.55)
 			(layers "F.Cu" "F.Mask" "F.Paste")
-			(net 22 "/PTT")
+			(net 25 "/TX_EN")
 			(pinfunction "PD4(XCK0/T0/PTCXY)")
 			(pintype "bidirectional")
@@
 			(size 1.6 0.55)
 			(layers "F.Cu" "F.Mask" "F.Paste")
-			(net 34 "/B0")
+			(net 45 "unconnected-(U1-PE0(SDA1{slash}ICP4{slash}ACO{slash}PTCXY)-Pad3)")
 			(pinfunction "PE0(SDA1/ICP4/ACO/PTCXY)")
-			(pintype "bidirectional")
+			(pintype "bidirectional+no_connect")
 			(solder_mask_margin 0.102)
 		)
@@
 			(size 1.6 0.55)
 			(layers "F.Cu" "F.Mask" "F.Paste")
-			(net 36 "/B1")
+			(net 40 "unconnected-(U1-PE1(SCL1{slash}T4{slash}PTCXY)-Pad6)")
 			(pinfunction "PE1(SCL1/T4/PTCXY)")
-			(pintype "bidirectional")
+			(pintype "bidirectional+no_connect")
 			(solder_mask_margin 0.102)
 		)
@@
 			(size 1.6 0.55)
 			(layers "F.Cu" "F.Mask" "F.Paste")
-			(net 37 "/B2")
+			(net 32 "unconnected-(U1-PE2(ADC6{slash}PTCY{slash}ICP3{slash}~{SS1})-Pad19)")
 			(pinfunction "PE2(ADC6/PTCY/ICP3/~{SS1})")
-			(pintype "bidirectional")
+			(pintype "bidirectional+no_connect")
 			(solder_mask_margin 0.102)
 		)
@@
 			(size 1.6 0.55)
 			(layers "F.Cu" "F.Mask" "F.Paste")
-			(net 38 "/B3")
+			(net 41 "unconnected-(U1-PE3(ADC7{slash}PTCY{slash}T3{slash}MOSI1)-Pad22)")
 			(pinfunction "PE3(ADC7/PTCY/T3/MOSI1)")
-			(pintype "bidirectional")
+			(pintype "bidirectional+no_connect")
 			(solder_mask_margin 0.102)
 		)
@@
 			(size 1.6 0.55)
 			(layers "F.Cu" "F.Mask" "F.Paste")
-			(net 25 "unconnected-(U1-PC0(ADC0{slash}PTCY{slash}MISO1)-Pad23)")
+			(net 34 "/B0")
 			(pinfunction "PC0(ADC0/PTCY/MISO1)")
-			(pintype "bidirectional+no_connect")
+			(pintype "bidirectional")
 			(solder_mask_margin 0.102)
 		)
@@
 			(size 1.6 0.55)
 			(layers "F.Cu" "F.Mask" "F.Paste")
-			(net 32 "unconnected-(U1-PC1(ADC1{slash}PTCY{slash}SCK1)-Pad24)")
+			(net 36 "/B1")
 			(pinfunction "PC1(ADC1/PTCY/SCK1)")
-			(pintype "bidirectional+no_connect")
+			(pintype "bidirectional")
 			(solder_mask_margin 0.102)
 		)
@@
 			(size 0.55 1.6)
 			(layers "F.Cu" "F.Mask" "F.Paste")
-			(net 26 "unconnected-(U1-PC2(ADC2{slash}PTCY)-Pad25)")
+			(net 37 "/B2")
 			(pinfunction "PC2(ADC2/PTCY)")
-			(pintype "bidirectional+no_connect")
+			(pintype "bidirectional")
 			(solder_mask_margin 0.102)
 		)
@@
 			(size 0.55 1.6)
 			(layers "F.Cu" "F.Mask" "F.Paste")
-			(net 40 "/SD")
+			(net 38 "/B3")
 			(pinfunction "PC3(ADC3/PTCY)")
 			(pintype "bidirectional")
@@
 			(size 0.55 1.6)
 			(layers "F.Cu" "F.Mask" "F.Paste")
-			(net 16 "/RST")
+			(net 6 "/RESET")
 			(pinfunction "PC6(~{RESET})")
 			(pintype "bidirectional")
@@
 			(size 0.55 1.6)
 			(layers "F.Cu" "F.Mask" "F.Paste")
-			(net 6 "/AUDIO_IN")
+			(net 26 "/SQL")
 			(pinfunction "PD1(PTCXY/OC4A/TXD0)")
 			(pintype "bidirectional")
@@
 			(layers "F.Cu" "F.Mask" "F.Paste")
 			(roundrect_rratio 0.208333)
-			(net 22 "/PTT")
+			(net 16 "Net-(J9-Pin_2)")
 			(pintype "passive")
 		)
@@
 			(layers "F.Cu" "F.Mask" "F.Paste")
 			(roundrect_rratio 0.208333)
-			(net 41 "Net-(Q1-C)")
+			(net 22 "/PTT")
 			(pintype "passive")
 		)
@@
 			(layers "F.Cu" "F.Mask" "F.Paste")
 			(roundrect_rratio 0.208333)
-			(net 22 "/PTT")
+			(net 25 "/TX_EN")
 			(pintype "passive")
 		)
@@
 			(layers "*.Cu" "*.Mask")
 			(remove_unused_layers no)
-			(net 22 "/PTT")
+			(net 16 "Net-(J9-Pin_2)")
 			(pinfunction "Pin_2")
 			(pintype "passive")
@@
 			(layers "F.Cu" "F.Mask" "F.Paste")
 			(roundrect_rratio 0.25)
-			(net 41 "Net-(Q1-C)")
+			(net 22 "/PTT")
 			(pinfunction "C")
 			(pintype "passive")
@@
 			(layers "F.Cu" "F.Mask" "F.Paste")
 			(roundrect_rratio 0.208333)
-			(net 22 "/PTT")
+			(net 25 "/TX_EN")
 			(pintype "passive")
 		)
@@
 			(layers "B.Cu" "B.Mask" "B.Paste")
 			(roundrect_rratio 0.208333)
-			(net 16 "/RST")
+			(net 6 "/RESET")
 			(pintype "passive")
 		)
